Commit message: Sim launch dependant on vehicle name and fix on description of myellow

File: farol2_description/urdf/myellow.xacro (robot description, xacro)
@@ -2,9 +2,21 @@
 <robot xmlns:xacro="http://www.ros.org/wiki/xacro" name="myellow">
   <!-- Constants -->
-  <xacro:property name="M_PI"     value="3.1415926535897931" />
+  <xacro:property name="M_PI" value="3.1415926535897931" />
+  <!-- Materials -->
+  <material name="blue">
+    <color rgba="0 0 1 1"/>
+  </material>
   <!-- Base -->
   <link name="base_link"/>
   <!-- Portside horizontal back thruster -->
-  <link name="thruster_portside_horizontal_back_link"/>
+  <link name="thruster_portside_horizontal_back_link">
+    <visual>
+      <origin xyz="0 0 0" rpy="0 1.5708 0"/>
+      <geometry>
+        <cylinder radius="0.02" length="0.08"/>
+      </geometry>
+      <material name="blue"/>
+    </visual>
+  </link>
   <joint name="base_to_thruster_portside_horizontal_back" type="fixed">
     <parent link="base_link"/>
@@ -13,5 +25,13 @@
   </joint>
   <!-- Starboard horizontal back thruster -->
-  <link name="thruster_starboard_horizontal_back_link"/>
+  <link name="thruster_starboard_horizontal_back_link">
+    <visual>
+      <origin xyz="0 0 0" rpy="0 1.5708 0"/>
+      <geometry>
+        <cylinder radius="0.02" length="0.08"/>
+      </geometry>
+      <material name="blue"/>
+    </visual>
+  </link>
   <joint name="base_to_thruster_starboard_horizontal_back" type="fixed">
     <parent link="base_link"/>
@@ -20,19 +40,43 @@
   </joint>
   <!-- Portside vertical thruster -->
-  <link name="thruster_portside_vertical_link"/>
+  <link name="thruster_portside_vertical_link">
+    <visual>
+      <origin xyz="0 0 0" rpy="0 1.5708 0"/>
+      <geometry>
+        <cylinder radius="0.02" length="0.08"/>
+      </geometry>
+      <material name="blue"/>
+    </visual>
+  </link>
   <joint name="base_to_thruster_portside_vertical" type="fixed">
     <parent link="base_link"/>
-    <child link="thruster_portside_vertical_link"/>
+    <child link="thruster_starboard_vertical_link"/>
     <origin xyz="0.087 -0.120 -0.12" rpy="0 -${0.5*M_PI} 0"/>
   </joint>
   <!-- Starboard vertical thruster -->
-  <link name="thruster_starboard_vertical_link"/>
+  <link name="thruster_starboard_vertical_link">
+    <visual>
+      <origin xyz="0 0 0" rpy="0 1.5708 0"/>
+      <geometry>
+        <cylinder radius="0.02" length="0.08"/>
+      </geometry>
+      <material name="blue"/>
+    </visual>
+  </link>
   <joint name="base_to_thruster_starboard_vertical" type="fixed">
     <parent link="base_link"/>
-    <child link="thruster_starboard_vertical_link"/>
+    <child link="thruster_portside_vertical_link"/>
     <origin xyz="0.087 0.120 -0.12" rpy="0 -${0.5*M_PI} 0"/>
   </joint>
   <!-- Portside horizontal front thruster -->
-  <link name="thruster_portside_horizontal_front_link"/>
+  <link name="thruster_portside_horizontal_front_link">
+    <visual>
+      <origin xyz="0 0 0" rpy="0 1.5708 0"/>
+      <geometry>
+        <cylinder radius="0.02" length="0.08"/>
+      </geometry>
+      <material name="blue"/>
+    </visual>
+  </link>
   <joint name="base_to_thruster_portside_horizontal_front" type="fixed">
     <parent link="base_link"/>
@@ -41,5 +85,13 @@
   </joint>
   <!-- Starboard horizontal front thruster -->
-  <link name="thruster_starboard_horizontal_front_link"/>
+  <link name="thruster_starboard_horizontal_front_link">
+    <visual>
+      <origin xyz="0 0 0" rpy="0 1.5708 0"/>
+      <geometry>
+        <cylinder radius="0.02" length="0.08"/>
+      </geometry>
+      <material name="blue"/>
+    </visual>
+  </link>
   <joint name="base_to_thruster_starboard_horizontal_front" type="fixed">
     <parent link="base_link"/>
