Commit message: Added TF to allocation, simulation bringup, now dependant on the name of the vehicle

File: farol2_description/urdf/magicelectric.xacro (robot description, xacro)
@@ -12,6 +12,12 @@
     <origin xyz="0.0 0.0 0.0" rpy="0 0 0"/>
   </joint>
-  <!-- Thrusters -->
-  <!-- ! Right now Z location of thruters is the same as center of mass because its simulated that way in holoocean -->
+  <!-- Pseudo thruster (middle) -->
+  <link name="thruster_middle_link"/>
+  <joint name="base_to_thruster_middle" type="fixed">
+    <parent link="base_link"/>
+    <child link="thruster_middle_link"/>
+    <origin xyz="-0.5 0.0 0.0" rpy="0 0 0"/>
+  </joint>
+  <!-- Thrusters (commented out)
   <link name="thruster_left_link"/>
   <joint name="base_to_thruster_left" type="fixed">
@@ -26,3 +32,4 @@
     <origin xyz="-0.5 -0.34 0.0" rpy="0 0 0"/>
   </joint>
+  -->
 </robot>

Commit message: Added PID fo depth and altitude and added vehicles. Changed launch files

File: farol2_description/urdf/magicelectric.xacro (robot description, xacro)
@@ -17,5 +17,5 @@
     <parent link="base_link"/>
     <child link="thruster_middle_link"/>
-    <origin xyz="-0.5 0.0 0.0" rpy="0 0 0"/>
+    <origin xyz="-4.0 0.0 0.0" rpy="0 0 0"/>
   </joint>
   <!-- Thrusters (commented out)
@@ -24,5 +24,5 @@
     <parent link="base_link"/>
     <child link="thruster_left_link"/>
-    <origin xyz="-0.5 0.34 0.0" rpy="0 0 0"/>
+    <origin xyz="-4.0 -1.5 0.0" rpy="0 0 0"/>
   </joint>
   <link name="thruster_right_link"/>
@@ -30,5 +30,5 @@
     <parent link="base_link"/>
     <child link="thruster_right_link"/>
-    <origin xyz="-0.5 -0.34 0.0" rpy="0 0 0"/>
+    <origin xyz="-4.0 1.5 0.0" rpy="0 0 0"/>
   </joint>
   -->

File: farol2_description/urdf/mred.xacro (robot description, xacro)
@@ -5,16 +5,31 @@
   <!-- Base -->
   <link name="base_link"/>
-  <!-- Thrusters -->
-  <link name="thruster_portside_link"/>
-  <joint name="base_to_thruster_portside" type="fixed">
+  <!-- Portside horizontal thruster -->
+  <link name="thruster_portside_horizontal_link"/>
+  <joint name="base_to_thruster_portside_horizontal" type="fixed">
     <parent link="base_link"/>
-    <child link="thruster_portside_link"/>
-    <origin xyz="-0.25 -0.15 0.0" rpy="0 0 0"/>
+    <child link="thruster_portside_horizontal_link"/>
+    <origin xyz="-0.290 0.140 0.011" rpy="0 0 0"/>
   </joint>
-  <link name="thruster_starboard_link"/>
-  <joint name="base_to_thruster_starboard" type="fixed">
+  <!-- Starboard horizontal thruster -->
+  <link name="thruster_starboard_horizontal_link"/>
+  <joint name="base_to_thruster_starboard_horizontal" type="fixed">
     <parent link="base_link"/>
-    <child link="thruster_starboard_link"/>
-    <origin xyz="-0.25 0.15 0.0" rpy="0 0 0"/>
+    <child link="thruster_starboard_horizontal_link"/>
+    <origin xyz="-0.290 -0.140 0.011" rpy="0 0 0"/>
+  </joint>
+  <!-- Portside vertical thruster -->
+  <link name="thruster_portside_vertical_link"/>
+  <joint name="base_to_thruster_portside_vertical" type="fixed">
+    <parent link="base_link"/>
+    <child link="thruster_portside_vertical_link"/>
+    <origin xyz="-0.012 -0.140 -0.107" rpy="0 -${0.5*M_PI} 0"/>
+  </joint>
+  <!-- Starboard vertical thruster -->
+  <link name="thruster_starboard_vertical_link"/>
+  <joint name="base_to_thruster_starboard_vertical" type="fixed">
+    <parent link="base_link"/>
+    <child link="thruster_starboard_vertical_link"/>
+    <origin xyz="-0.012 0.140 -0.107" rpy="0 -${0.5*M_PI} 0"/>
   </joint>
 </robot>

File: farol2_description/urdf/myellow.xacro (robot description, xacro)
@@ -5,47 +5,45 @@
   <!-- Base -->
   <link name="base_link"/>
-  <!-- Thrusters -->
-  <link name="thruster_portside_bow"/>
-  <joint name="base_to_thruster_portside_bow" type="fixed">
+  <!-- Portside horizontal back thruster -->
+  <link name="thruster_portside_horizontal_back_link"/>
+  <joint name="base_to_thruster_portside_horizontal_back" type="fixed">
     <parent link="base_link"/>
-    <child link="thruster_portside_bow"/>
-    <origin xyz="-0.5 0.34 0.0" rpy="0 0 0"/>
+    <child link="thruster_portside_horizontal_back_link"/>
+    <origin xyz="-0.306 0.062 0.0" rpy="0 0 ${0.25*M_PI}"/>
   </joint>
-  <link name="thruster_portside_stern"/>
-  <joint name="base_to_thruster_portside_stern" type="fixed">
+  <!-- Starboard horizontal back thruster -->
+  <link name="thruster_starboard_horizontal_back_link"/>
+  <joint name="base_to_thruster_starboard_horizontal_back" type="fixed">
     <parent link="base_link"/>
-    <child link="thruster_portside_stern"/>
-    <origin xyz="0.5 0.34 0.0" rpy="0 0 0"/>
+    <child link="thruster_starboard_horizontal_back_link"/>
+    <origin xyz="-0.306 -0.062 0.0" rpy="0 0 -${0.25*M_PI}"/>
   </joint>
-  <link name="thruster_portside_vertical"/>
+  <!-- Portside vertical thruster -->
+  <link name="thruster_portside_vertical_link"/>
   <joint name="base_to_thruster_portside_vertical" type="fixed">
     <parent link="base_link"/>
-    <child link="thruster_portside_vertical"/>
-    <origin xyz="0.0 0.34 0.0" rpy="0 0 0"/>
+    <child link="thruster_portside_vertical_link"/>
+    <origin xyz="0.087 -0.120 -0.12" rpy="0 -${0.5*M_PI} 0"/>
   </joint>
-  <link name="thruster_starboard_bow"/>
-  <joint name="base_to_thruster_starboard_bow" type="fixed">
-    <parent link="base_link"/>
-    <child link="thruster_starboard_bow"/>
-    <origin xyz="0.5 -0.34 0.0" rpy="0 0 0"/>
-  </joint>
-  <link name="thruster_starboard_stern"/>
-  <joint name="base_to_thruster_starboard_stern" type="fixed">
-    <parent link="base_link"/>
-    <child link="thruster_starboard_stern"/>
-    <origin xyz="-0.5 -0.34 0.0" rpy="0 0 0"/>
-  </joint>
-  <link name="thruster_starboard_vertical"/>
+  <!-- Starboard vertical thruster -->
+  <link name="thruster_starboard_vertical_link"/>
   <joint name="base_to_thruster_starboard_vertical" type="fixed">
     <parent link="base_link"/>
-    <child link="thruster_starboard_vertical"/>
-    <origin xyz="0.0 -0.34 0.0" rpy="0 0 0"/>
+    <child link="thruster_starboard_vertical_link"/>
+    <origin xyz="0.087 0.120 -0.12" rpy="0 -${0.5*M_PI} 0"/>
   </joint>
-  <!-- IMU -->
-  <link name="imu_link"/>
-  <joint name="base_to_imu" type="fixed">
+  <!-- Portside horizontal front thruster -->
+  <link name="thruster_portside_horizontal_front_link"/>
+  <joint name="base_to_thruster_portside_horizontal_front" type="fixed">
     <parent link="base_link"/>
-    <child link="imu_link"/>
-    <origin xyz="0.0 0.0 0.0" rpy="0 0 0"/>
+    <child link="thruster_portside_horizontal_front_link"/>
+    <origin xyz="0.300 0.197 0.0" rpy="0 0 -${0.25*M_PI}"/>
+  </joint>
+  <!-- Starboard horizontal front thruster -->
+  <link name="thruster_starboard_horizontal_front_link"/>
+  <joint name="base_to_thruster_starboard_horizontal_front" type="fixed">
+    <parent link="base_link"/>
+    <child link="thruster_starboard_horizontal_front_link"/>
+    <origin xyz="0.300 -0.197 0.0" rpy="0 0 ${0.25*M_PI}"/>
   </joint>
 </robot>

Commit message: Added clock node to allow several simulation launches at the same time. Added dynamic TF for rudder in Magic Electric.

File: farol2_description/urdf/magicelectric.xacro (robot description, xacro)
@@ -2,14 +2,7 @@
 <robot xmlns:xacro="http://www.ros.org/wiki/xacro" name="magicelectric">
   <!-- Constants -->
-  <xacro:property name="M_PI"     value="3.1415926535897931" />
+  <xacro:property name="M_PI" value="3.1415926535897931" />
   <!-- Base -->
   <link name="base_link"/>
-  <!-- INS -->
-  <link name="ins_link"/>
-  <joint name="base_to_ins" type="fixed">
-    <parent link="base_link"/>
-    <child link="ins_link"/>
-    <origin xyz="0.0 0.0 0.0" rpy="0 0 0"/>
-  </joint>
   <!-- Pseudo thruster (middle) -->
   <link name="thruster_middle_link"/>
@@ -19,5 +12,13 @@
     <origin xyz="-4.0 0.0 0.0" rpy="0 0 0"/>
   </joint>
-  <!-- Thrusters (commented out)
+  <!-- Pseudo rudder (middle, dynamic rotation) -->
+  <link name="rudder_middle_link"/>
+  <joint name="base_to_rudder_middle" type="continuous">
+    <parent link="base_link"/>
+    <child link="rudder_middle_link"/>
+    <origin xyz="-4.5 0.0 0.0" rpy="0 0 ${1*M_PI}"/>
+    <axis xyz="0 0 1"/>
+  </joint>
+  <!-- Thrusters and rudders
   <link name="thruster_left_link"/>
   <joint name="base_to_thruster_left" type="fixed">
@@ -32,4 +33,18 @@
     <origin xyz="-4.0 1.5 0.0" rpy="0 0 0"/>
   </joint>
+  <link name="rudder_left_link"/>
+  <joint name="base_to_rudder_left" type="continuous">
+    <parent link="base_link"/>
+    <child link="rudder_left_link"/>
+    <origin xyz="-4.5 -1.5 0.0" rpy="0 0 0"/>
+    <axis xyz="0 0 1"/>
+  </joint>
+  <link name="rudder_right_link"/>
+  <joint name="base_to_rudder_right" type="continuous">
+    <parent link="base_link"/>
+    <child link="rudder_right_link"/>
+    <origin xyz="-4.5 1.5 0.0" rpy="0 0 0"/>
+    <axis xyz="0 0 1"/>
+  </joint>
   -->
 </robot>

Commit message: Changed vehicle description format

File: farol2_description/urdf/magicelectric.xacro (robot description, xacro)
@@ -3,48 +3,52 @@
   <!-- Constants -->
   <xacro:property name="M_PI" value="3.1415926535897931" />
+  <xacro:arg name="simple_allocation" default="true" />
   <!-- Base -->
   <link name="base_link"/>
-  <!-- Pseudo thruster (middle) -->
-  <link name="thruster_middle_link"/>
-  <joint name="base_to_thruster_middle" type="fixed">
-    <parent link="base_link"/>
-    <child link="thruster_middle_link"/>
-    <origin xyz="-4.0 0.0 0.0" rpy="0 0 0"/>
-  </joint>
-  <!-- Pseudo rudder (middle, dynamic rotation) -->
-  <link name="rudder_middle_link"/>
-  <joint name="base_to_rudder_middle" type="continuous">
-    <parent link="base_link"/>
-    <child link="rudder_middle_link"/>
-    <origin xyz="-4.5 0.0 0.0" rpy="0 0 ${1*M_PI}"/>
-    <axis xyz="0 0 1"/>
-  </joint>
-  <!-- Thrusters and rudders
-  <link name="thruster_left_link"/>
-  <joint name="base_to_thruster_left" type="fixed">
-    <parent link="base_link"/>
-    <child link="thruster_left_link"/>
-    <origin xyz="-4.0 -1.5 0.0" rpy="0 0 0"/>
-  </joint>
-  <link name="thruster_right_link"/>
-  <joint name="base_to_thruster_right" type="fixed">
-    <parent link="base_link"/>
-    <child link="thruster_right_link"/>
-    <origin xyz="-4.0 1.5 0.0" rpy="0 0 0"/>
-  </joint>
-  <link name="rudder_left_link"/>
-  <joint name="base_to_rudder_left" type="continuous">
-    <parent link="base_link"/>
-    <child link="rudder_left_link"/>
-    <origin xyz="-4.5 -1.5 0.0" rpy="0 0 0"/>
-    <axis xyz="0 0 1"/>
-  </joint>
-  <link name="rudder_right_link"/>
-  <joint name="base_to_rudder_right" type="continuous">
-    <parent link="base_link"/>
-    <child link="rudder_right_link"/>
-    <origin xyz="-4.5 1.5 0.0" rpy="0 0 0"/>
-    <axis xyz="0 0 1"/>
-  </joint>
-  -->
+  <xacro:if value="$(arg simple_allocation)">
+    <!-- Pseudo thruster (middle) -->
+    <link name="thruster_middle_link"/>
+    <joint name="base_to_thruster_middle" type="fixed">
+      <parent link="base_link"/>
+      <child link="thruster_middle_link"/>
+      <origin xyz="-4.0 0.0 0.0" rpy="0 0 0"/>
+    </joint>
+    <!-- Pseudo rudder (middle, dynamic rotation) -->
+    <link name="rudder_middle_link"/>
+    <joint name="base_to_rudder_middle" type="continuous">
+      <parent link="base_link"/>
+      <child link="rudder_middle_link"/>
+      <origin xyz="-4.5 0.0 0.0" rpy="0 0 ${1*M_PI}"/>
+      <axis xyz="0 0 1"/>
+    </joint>
+  </xacro:if>
+  <xacro:unless value="$(arg simple_allocation)">
+    <!-- Thrusters and rudders -->
+    <link name="thruster_left_link"/>
+    <joint name="base_to_thruster_left" type="fixed">
+      <parent link="base_link"/>
+      <child link="thruster_left_link"/>
+      <origin xyz="-4.0 -1.5 0.0" rpy="0 0 0"/>
+    </joint>
+    <link name="thruster_right_link"/>
+    <joint name="base_to_thruster_right" type="fixed">
+      <parent link="base_link"/>
+      <child link="thruster_right_link"/>
+      <origin xyz="-4.0 1.5 0.0" rpy="0 0 0"/>
+    </joint>
+    <link name="rudder_left_link"/>
+    <joint name="base_to_rudder_left" type="continuous">
+      <parent link="base_link"/>
+      <child link="rudder_left_link"/>
+      <origin xyz="-4.5 -1.5 0.0" rpy="0 0 0"/>
+      <axis xyz="0 0 1"/>
+    </joint>
+    <link name="rudder_right_link"/>
+    <joint name="base_to_rudder_right" type="continuous">
+      <parent link="base_link"/>
+      <child link="rudder_right_link"/>
+      <origin xyz="-4.5 1.5 0.0" rpy="0 0 0"/>
+      <axis xyz="0 0 1"/>
+    </joint>
+  </xacro:unless>
 </robot>

File: farol2_description/urdf/myellow.xacro (robot description, xacro)
@@ -3,20 +3,8 @@
   <!-- Constants -->
   <xacro:property name="M_PI" value="3.1415926535897931" />
-  <!-- Materials -->
-  <material name="blue">
-    <color rgba="0 0 1 1"/>
-  </material>
   <!-- Base -->
   <link name="base_link"/>
   <!-- Portside horizontal back thruster -->
-  <link name="thruster_portside_horizontal_back_link">
-    <visual>
-      <origin xyz="0 0 0" rpy="0 1.5708 0"/>
-      <geometry>
-        <cylinder radius="0.02" length="0.08"/>
-      </geometry>
-      <material name="blue"/>
-    </visual>
-  </link>
+  <link name="thruster_portside_horizontal_back_link"/>
   <joint name="base_to_thruster_portside_horizontal_back" type="fixed">
     <parent link="base_link"/>
@@ -25,13 +13,5 @@
   </joint>
   <!-- Starboard horizontal back thruster -->
-  <link name="thruster_starboard_horizontal_back_link">
-    <visual>
-      <origin xyz="0 0 0" rpy="0 1.5708 0"/>
-      <geometry>
-        <cylinder radius="0.02" length="0.08"/>
-      </geometry>
-      <material name="blue"/>
-    </visual>
-  </link>
+  <link name="thruster_starboard_horizontal_back_link"/>
   <joint name="base_to_thruster_starboard_horizontal_back" type="fixed">
     <parent link="base_link"/>
@@ -40,13 +20,5 @@
   </joint>
   <!-- Portside vertical thruster -->
-  <link name="thruster_portside_vertical_link">
-    <visual>
-      <origin xyz="0 0 0" rpy="0 1.5708 0"/>
-      <geometry>
-        <cylinder radius="0.02" length="0.08"/>
-      </geometry>
-      <material name="blue"/>
-    </visual>
-  </link>
+  <link name="thruster_portside_vertical_link"/>
   <joint name="base_to_thruster_portside_vertical" type="fixed">
     <parent link="base_link"/>
@@ -55,13 +27,5 @@
   </joint>
   <!-- Starboard vertical thruster -->
-  <link name="thruster_starboard_vertical_link">
-    <visual>
-      <origin xyz="0 0 0" rpy="0 1.5708 0"/>
-      <geometry>
-        <cylinder radius="0.02" length="0.08"/>
-      </geometry>
-      <material name="blue"/>
-    </visual>
-  </link>
+  <link name="thruster_starboard_vertical_link"/>
   <joint name="base_to_thruster_starboard_vertical" type="fixed">
     <parent link="base_link"/>
@@ -70,13 +34,5 @@
   </joint>
   <!-- Portside horizontal front thruster -->
-  <link name="thruster_portside_horizontal_front_link">
-    <visual>
-      <origin xyz="0 0 0" rpy="0 1.5708 0"/>
-      <geometry>
-        <cylinder radius="0.02" length="0.08"/>
-      </geometry>
-      <material name="blue"/>
-    </visual>
-  </link>
+  <link name="thruster_portside_horizontal_front_link"/>
   <joint name="base_to_thruster_portside_horizontal_front" type="fixed">
     <parent link="base_link"/>
@@ -85,13 +41,5 @@
   </joint>
   <!-- Starboard horizontal front thruster -->
-  <link name="thruster_starboard_horizontal_front_link">
-    <visual>
-      <origin xyz="0 0 0" rpy="0 1.5708 0"/>
-      <geometry>
-        <cylinder radius="0.02" length="0.08"/>
-      </geometry>
-      <material name="blue"/>
-    </visual>
-  </link>
+  <link name="thruster_starboard_horizontal_front_link"/>
   <joint name="base_to_thruster_starboard_horizontal_front" type="fixed">
     <parent link="base_link"/>
