Commit message: config changes and small allocation bringup cleanup

File: farol2_description/urdf/bluerov.xacro (robot description, xacro)
@@ -10,5 +10,5 @@
     <parent link="base_link"/>
     <child link="thruster_starboard_horizontal_front_link"/>
-    <origin xyz="0.1355 -0.1 -0.0725" rpy="0 0 ${0.25*M_PI}"/>
+    <origin xyz="0.1355 0.1 -0.0725" rpy="0 0 ${0.25*M_PI}"/>
   </joint>
   <!-- Portside horizontal front thruster -->
@@ -17,5 +17,5 @@
     <parent link="base_link"/>
     <child link="thruster_portside_horizontal_front_link"/>
-    <origin xyz="0.1355 0.1 -0.0725" rpy="0 0 -${0.25*M_PI}"/>
+    <origin xyz="0.1355 -0.1 -0.0725" rpy="0 0 -${0.25*M_PI}"/>
   </joint>
   <!-- Starboard horizontal back thruster -->
@@ -24,5 +24,5 @@
     <parent link="base_link"/>
     <child link="thruster_starboard_horizontal_back_link"/>
-    <origin xyz="-0.1475 -0.1 -0.0725" rpy="0 0 ${0.75*M_PI}"/>
+    <origin xyz="-0.1475 0.1 -0.0725" rpy="0 0 ${0.75*M_PI}"/>
   </joint>
   <!-- Portside horizontal back thruster -->
@@ -31,5 +31,5 @@
     <parent link="base_link"/>
     <child link="thruster_portside_horizontal_back_link"/>
-    <origin xyz="-0.1475 0.1 -0.0725" rpy="0 0 -${0.75*M_PI}"/>
+    <origin xyz="-0.1475 -0.1 -0.0725" rpy="0 0 -${0.75*M_PI}"/>
   </joint>
   <!-- Starboard vertical front thruster -->
@@ -38,5 +38,5 @@
     <parent link="base_link"/>
     <child link="thruster_starboard_vertical_front_link"/>
-    <origin xyz="0.12 -0.22 -0.005" rpy="0 -${0.5*M_PI} 0"/>
+    <origin xyz="0.12 0.22 -0.005" rpy="0 -${0.5*M_PI} 0"/>
   </joint>
   <!-- Portside vertical front thruster -->
@@ -45,5 +45,5 @@
     <parent link="base_link"/>
     <child link="thruster_portside_vertical_front_link"/>
-    <origin xyz="0.12 0.22 -0.005" rpy="0 -${0.5*M_PI} 0"/>
+    <origin xyz="0.12 -0.22 -0.005" rpy="0 -${0.5*M_PI} 0"/>
   </joint>
   <!-- Starboard vertical back thruster -->
@@ -52,5 +52,5 @@
     <parent link="base_link"/>
     <child link="thruster_starboard_vertical_back_link"/>
-    <origin xyz="-0.12 -0.22 -0.005" rpy="0 -${0.5*M_PI} 0"/>
+    <origin xyz="-0.12 0.22 -0.005" rpy="0 -${0.5*M_PI} 0"/>
   </joint>
   <!-- Portside vertical back thruster -->
@@ -59,5 +59,5 @@
     <parent link="base_link"/>
     <child link="thruster_portside_vertical_back_link"/>
-    <origin xyz="-0.12 0.22 -0.005" rpy="0 -${0.5*M_PI} 0"/>
+    <origin xyz="-0.12 -0.22 -0.005" rpy="0 -${0.5*M_PI} 0"/>
   </joint>
 </robot>

File: farol2_description/urdf/mblack.xacro (robot description, xacro)
@@ -10,5 +10,5 @@
     <parent link="base_link"/>
     <child link="thruster_portside_link"/>
-    <origin xyz="-0.29 0.14 0.0" rpy="0 0 0"/>
+    <origin xyz="-0.29 -0.14 0.0" rpy="0 0 0"/>
   </joint>
   <link name="thruster_starboard_link"/>
@@ -16,5 +16,5 @@
     <parent link="base_link"/>
     <child link="thruster_starboard_link"/>
-    <origin xyz="-0.29 -0.14 0.0" rpy="0 0 0"/>
+    <origin xyz="-0.29 0.14 0.0" rpy="0 0 0"/>
   </joint>
 </robot>

File: farol2_description/urdf/myellow.xacro (robot description, xacro)
@@ -10,5 +10,5 @@
     <parent link="base_link"/>
     <child link="thruster_portside_horizontal_back_link"/>
-    <origin xyz="-0.306 0.062 0.0" rpy="0 0 ${0.25*M_PI}"/>
+    <origin xyz="-0.306 -0.062 0.0" rpy="0 0 ${0.25*M_PI}"/>
   </joint>
   <!-- Starboard horizontal back thruster -->
@@ -17,5 +17,5 @@
     <parent link="base_link"/>
     <child link="thruster_starboard_horizontal_back_link"/>
-    <origin xyz="-0.306 -0.062 0.0" rpy="0 0 -${0.25*M_PI}"/>
+    <origin xyz="-0.306 0.062 0.0" rpy="0 0 -${0.25*M_PI}"/>
   </joint>
   <!-- Portside vertical thruster -->
@@ -24,5 +24,5 @@
     <parent link="base_link"/>
     <child link="thruster_starboard_vertical_link"/>
-    <origin xyz="0.087 -0.120 -0.12" rpy="0 -${0.5*M_PI} 0"/>
+    <origin xyz="0.087 0.120 -0.12" rpy="0 -${0.5*M_PI} 0"/>
   </joint>
   <!-- Starboard vertical thruster -->
@@ -31,5 +31,5 @@
     <parent link="base_link"/>
     <child link="thruster_portside_vertical_link"/>
-    <origin xyz="0.087 0.120 -0.12" rpy="0 -${0.5*M_PI} 0"/>
+    <origin xyz="0.087 -0.120 -0.12" rpy="0 -${0.5*M_PI} 0"/>
   </joint>
   <!-- Portside horizontal front thruster -->
@@ -38,5 +38,5 @@
     <parent link="base_link"/>
     <child link="thruster_portside_horizontal_front_link"/>
-    <origin xyz="0.300 0.197 0.0" rpy="0 0 -${0.25*M_PI}"/>
+    <origin xyz="0.300 -0.197 0.0" rpy="0 0 -${0.25*M_PI}"/>
   </joint>
   <!-- Starboard horizontal front thruster -->
@@ -45,5 +45,5 @@
     <parent link="base_link"/>
     <child link="thruster_starboard_horizontal_front_link"/>
-    <origin xyz="0.300 -0.197 0.0" rpy="0 0 ${0.25*M_PI}"/>
+    <origin xyz="0.300 0.197 0.0" rpy="0 0 ${0.25*M_PI}"/>
   </joint>
 </robot>
